File: kicad/basic-bbb-cape.kicad_pcb (KiCad board)
At the start: 2 copper layers, 54.6 x 86.4 mm, 6 parts, among them P1 BeagleBone_Black_Header, P2 BeagleBone_Black_Header, U1 CAT24C32YI-GT3

Commit message: Update schematic and PCB
Parts:
- RN1: value 5.6 k -> R_Pack07
- moved JP1 14.6 mm to (118.3, 49.7)
- moved RN1 13.9 mm to (125.2, 45.3), turned to 0 degrees
- moved JP2 13.6 mm to (118.2, 54.8)
- moved U1 0.60 mm to (130.1, 68.1)
Connections:
- RN1 pad 1: Net-(JP1-Pad2) -> +3V3
- RN1 pad 10: +3V3 -> Net-(RN1-Pad10)
- RN1 pad 11: +3V3 -> Net-(RN1-Pad11)
- RN1 pad 12: +3V3 -> Net-(JP2-Pad2)
- RN1 pad 13: +3V3 -> Net-(JP1-Pad2)
- RN1 pad 14: +3V3 -> unconnected-(RN1-Pad14)
- RN1 pad 2: Net-(JP2-Pad2) -> +3V3
- RN1 pad 3: Net-(RN1-Pad3) -> +3V3
- RN1 pad 4: unconnected-(RN1-Pad4) -> +3V3
- RN1 pad 5: Net-(RN1-Pad5) -> +3V3
- RN1 pad 6: I2C2_SDA -> +3V3
- RN1 pad 7: I2C2_SCL -> +3V3
- RN1 pad 8: +3V3 -> I2C2_SCL
- RN1 pad 9: +3V3 -> I2C2_SDA
- U1 pad 3: Net-(RN1-Pad3) -> Net-(RN1-Pad11)
- U1 pad 7: Net-(RN1-Pad5) -> Net-(RN1-Pad10)

Commit message: Move RP1 socket
Parts:
- moved RN1 2.20 mm to (123.0, 45.3)
Changed lines of the file:
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@@
   )
   (footprint "Package_DIP:DIP-14_W7.62mm_Socket_LongPads" (layer "F.Cu")
-    (at 125.1701 45.2974)
+    (at 122.9701 45.2974)
     (descr "14-lead though-hole mounted DIP package, row spacing 7.62 mm (300 mils), Socket, LongPads")
     (tags "THT DIP DIL PDIP 2.54mm 7.62mm 300mil Socket LongPads")

Commit message: Resize schematic to 8x11 inch and reset PCH closer to defaults
Routing:
- net +3V3: track 14.6 -> 2.54 mm
- net unconnected-(P1-Pad23): track 8.16 -> 0.00 mm
- net unconnected-(P1-Pad17): track 4.08 -> 0.00 mm
- net unconnected-(P1-Pad21): track 3.60 -> 0.00 mm
- net unconnected-(P2-Pad13): track 2.81 -> 0.00 mm
- net unconnected-(P1-Pad16): track 2.19 -> 0.00 mm
- net unconnected-(P2-Pad18): track 1.91 -> 0.00 mm
- net unconnected-(P2-Pad19): track 1.78 -> 0.00 mm
- net unconnected-(P1-Pad15): track 1.68 -> 0.00 mm
- net unconnected-(P1-Pad14): track 1.52 -> 0.00 mm
- net unconnected-(P2-Pad17): track 1.27 -> 0.00 mm
Changed lines of the file:
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@@
     (effects (font (size 0.8 0.8) (thickness 0.14)) (justify left))
   )
-  (segment (start 115.506501 65.785999) (end 116.3701 64.9224) (width 0.25) (layer "B.Cu") (net 1))
-  (segment (start 115.799571 76.271001) (end 115.181499 75.652929) (width 0.25) (layer "B.Cu") (net 1))
-  (segment (start 115.181499 75.652929) (end 115.181499 66.111001) (width 0.25) (layer "B.Cu") (net 1))
-  (segment (start 115.181499 66.111001) (end 115.506501 65.785999) (width 0.25) (layer "B.Cu") (net 1))
   (segment (start 118.9101 64.9224) (end 116.3701 64.9224) (width 0.25) (layer "B.Cu") (net 1))
   (segment (start 116.3701 67.4624) (end 118.9101 67.4624) (width 1) (layer "B.Cu") (net 2))
   (segment (start 116.3701 70.0024) (end 118.9101 70.0024) (width 0.25) (layer "F.Cu") (net 3))
-  (segment (start 118.9101 77.6224) (end 120.4341 77.6224) (width 0.25) (layer "B.Cu") (net 10))
-  (segment (start 117.233699 81.025999) (end 116.3701 80.1624) (width 0.25) (layer "F.Cu") (net 11))
-  (segment (start 117.558701 81.351001) (end 117.233699 81.025999) (width 0.25) (layer "F.Cu") (net 11))
-  (segment (start 118.9101 80.1624) (end 120.098701 81.351001) (width 0.25) (layer "B.Cu") (net 12))
-  (segment (start 120.098701 81.351001) (end 120.098701 81.858003) (width 0.25) (layer "B.Cu") (net 12))
-  (segment (start 117.558701 83.891001) (end 117.233699 83.565999) (width 0.25) (layer "F.Cu") (net 13))
-  (segment (start 117.233699 83.565999) (end 116.3701 82.7024) (width 0.25) (layer "F.Cu") (net 13))
-  (segment (start 119.480629 83.891001) (end 117.558701 83.891001) (width 0.25) (layer "F.Cu") (net 13))
-  (segment (start 119.816028 84.2264) (end 119.480629 83.891001) (width 0.25) (layer "F.Cu") (net 13))
-  (segment (start 119.480629 88.971001) (end 117.558701 88.971001) (width 0.25) (layer "F.Cu") (net 17))
-  (segment (start 117.558701 88.971001) (end 117.233699 88.645999) (width 0.25) (layer "F.Cu") (net 17))
-  (segment (start 117.233699 88.645999) (end 116.3701 87.7824) (width 0.25) (layer "F.Cu") (net 17))
-  (segment (start 115.181499 93.432929) (end 115.181499 91.511001) (width 0.25) (layer "F.Cu") (net 19))
-  (segment (start 119.480629 94.051001) (end 115.799571 94.051001) (width 0.25) (layer "F.Cu") (net 19))
-  (segment (start 115.799571 94.051001) (end 115.181499 93.432929) (width 0.25) (layer "F.Cu") (net 19))
-  (segment (start 115.181499 91.511001) (end 115.506501 91.185999) (width 0.25) (layer "F.Cu") (net 19))
-  (segment (start 115.506501 91.185999) (end 116.3701 90.3224) (width 0.25) (layer "F.Cu") (net 19))
-  (segment (start 164.3761 72.2884) (end 164.6301 72.5424) (width 0.25) (layer "F.Cu") (net 43))
-  (segment (start 164.6301 77.6224) (end 162.643099 79.609401) (width 0.25) (layer "F.Cu") (net 47))
-  (segment (start 164.6301 82.7024) (end 163.728711 83.603789) (width 0.25) (layer "B.Cu") (net 51))
-  (segment (start 166.306501 83.565999) (end 167.1701 82.7024) (width 0.25) (layer "B.Cu") (net 52))
-  (segment (start 165.818701 84.053799) (end 166.306501 83.565999) (width 0.25) (layer "B.Cu") (net 52))
-  (segment (start 164.6301 85.2424) (end 162.8521 85.2424) (width 0.25) (layer "F.Cu") (net 53))
   (zone (net 4) (net_name "Earth") (layer "F.Cu") (hatch edge 0.508)
     (connect_pads (clearance 0.508))
-    (min_thickness 0.254)
+    (min_thickness 0.254) (filled_areas_thickness no)
     (fill yes (thermal_gap 0.508) (thermal_bridge_width 0.508))
     (polygon
@@
   (zone (net 4) (net_name "Earth") (layer "B.Cu") (hatch edge 0.508)
     (connect_pads (clearance 0.508))
-    (min_thickness 0.254)
+    (min_thickness 0.254) (filled_areas_thickness no)
     (fill yes (thermal_gap 0.508) (thermal_bridge_width 0.508))
     (polygon
